Commit message: kinetic

File: rom2109_description/urdf/rom2109_description.urdf (robot description, URDF)
Before this commit: robot rom2109, 8 links, 7 joints
Links:
- removed link plate2
- removed link plate3
- link base_link: mass 2.41256345237752 -> 2.3522
- link camera: mass 0.0447522001138537 -> 0.044752
- link left_wheel: mass 2.88257784807586 -> 2.8826
- link lidar: mass 1.33076913637071 -> 1.3308
- link plate1: mass 0.376303345586596 -> 0.3763
- link right_wheel: mass 2.88257784610314 -> 2.8826
Joints:
- removed joint plate2_joint
- removed joint plate3_joint
- joint camera_joint: origin xyz=0.1095 0.00557736269756118 -0.0125000000000011 rpy=0 0 0 -> xyz=0.1095 0.0055774 -0.0125 rpy=0 0 0
- joint lidar_joint: origin xyz=0.0159981253913104 -0.00158018301594729 0.0325999999999999 rpy=0 0 0 -> xyz=0.015998 -0.0015802 0.0326 rpy=0 0 0
- joint plate1_joint: origin xyz=-0.0038733 0 0.15505 rpy=0 0 0 -> xyz=-0.0038733 0 0.13505 rpy=0 0 0
