Commit message: urdf done, gz err

File: rom2109_description/urdf/rom2109_bot_gazebo11.urdf (robot description, URDF)
Before this commit: robot rom2109_description, 6 links, 5 joints
Links:
- link base_link: geometry collision mesh filename=model://rom2109_description/meshes/bot/base_link.STL; visual mesh filename=model://rom2109_description/meshes/bot/base_link.STL
- link frame_link: geometry collision mesh filename=model://rom2109_description/meshes/bot/frame_link.STL; visual mesh filename=model://rom2109_description/meshes/bot/frame_link.STL
- link left_wheel: geometry collision mesh filename=model://rom2109_description/meshes/bot/left_wheel.STL; visual mesh filename=model://rom2109_description/meshes/bot/left_wheel.STL
- link right_wheel: geometry collision mesh filename=model://rom2109_description/meshes/bot/right_wheel.STL; visual mesh filename=model://rom2109_description/meshes/bot/right_wheel.STL
- link rp_lidar: geometry collision mesh filename=model://rom2109_description/meshes/bot/rp_lidar.STL; visual mesh filename=model://rom2109_description/meshes/bot/rp_lidar.STL
- link wifi: geometry collision mesh filename=model://rom2109_description/meshes/bot/wifi.STL; visual mesh filename=model://rom2109_description/meshes/bot/wifi.STL
